File: tusb2036-demo.kicad_pcb (KiCad board)
At the start: 2 copper layers, 85 x 52 mm, 48 parts, among them J1 USB_B_Micro, J2 USB_A, J3 USB_A, J4 USB_A, SW1 RESET, U1 TUSB2036, U2 TPS76333, U3 TPS2044D, U4 SN75240, U5 SN75240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

Commit message: Fix 120uF caps
Parts:
- C20, C30, C40: footprint Capacitor_SMD:C_1206_3216Metric -> Vishay-cap:CAPPM7343X310N
- moved C30 54.1 mm to (135.2, 103.6), turned to 90 degrees
- moved C20 54.1 mm to (111.2, 103.6), turned to 90 degrees
- moved C40 54.1 mm to (159.2, 103.7), turned to 90 degrees
- moved J1 48.3 mm to (103.4, 122.0)
- moved U4 48.3 mm to (110.8, 115.1)
- moved C1 48.3 mm to (115.3, 84.2)
- moved C10 48.3 mm to (106.8, 107.7)
- moved C11 48.3 mm to (99.8, 107.7)
- moved C2 48.3 mm to (122.2, 84.2)
- moved C21 48.3 mm to (129.3, 99.2)
- moved C22 48.3 mm to (116.2, 99.2)
- moved C3 48.3 mm to (103.8, 93.7)
- moved C31 48.3 mm to (153.3, 99.2)
- moved C32 48.3 mm to (140.3, 99.2)
- moved C4 48.3 mm to (99.8, 93.7)
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Routing:
- net /5VB: track 35.3 -> 41.6 mm
- net /5VC: track 36.2 -> 42.4 mm
- net /5VA: track 49.1 -> 55.1 mm
Other:
- board text added: "TUSB2036 USB Hub Evaluation Board v2 C. Keller 2021-03-20"
- board text removed: "TUSB2036 USB Hub Evaluation Board v1 C. Keller 2021-03-20"
