File: tusb2036-eval.kicad_pcb (KiCad board)
At the start: 2 copper layers, 85 x 52 mm, 49 parts, among them J1 USB_B_Micro, J2 USB_A, J3 USB_A, J4 USB_A, SW1 RESET, U1 TUSB2036, U2 TPS76333, U3 TPS2044D, U4 SN75240, U5 SN75240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

Commit message: Add CC-BY-4.0 license
Other:
- board text added: "https://github.com/k0swe/tusb2036-eval"

Commit message: Fix up libraries
Parts:
- C20, C30, C40: footprint Vishay-cap:CAPPM7343X310N -> Vishay:CAPPM7343X310N
- J2, J3, J4: footprint USB-A:62900416021 -> Wurth:62900416021
- moved U4 0.14 mm to (110.8, 115.2)
- moved U3 0.06 mm to (154.2, 88.8)
Routing:
- net Net-(J2-Pad3): track 35.6 -> 29.6 mm
- net GND: track 138.2 -> 133.1 mm
- net Net-(J2-Pad2): track 29.0 -> 26.0 mm
- net /EN2: track 22.8 -> 20.4 mm

Commit message: Replace micro USB connector
The Molex is difficult to hand solder, so swapping that out for the CUI
Parts:
- J1: footprint Connector_USB:USB_Micro-B_Molex_47346-0001 -> CUI:UJ2-MIBH-4-SMT
- moved R10 5.76 mm to (104.0, 109.0)
- moved R11 5.72 mm to (101.5, 109.0)
- moved C11 3.31 mm to (99.0, 104.5)
- moved C10 3.23 mm to (106.5, 104.5)
- moved J1 3.20 mm to (103.2, 125.2), turned to 180 degrees
Connections:
- net Net-(J1-Pad2) renamed /U0-
- net Net-(J1-Pad3) renamed /U0+
- net Net-(J2-Pad2) renamed /U1-
- net Net-(J2-Pad3) renamed /U1+
- net Net-(J3-Pad2) renamed /U2-
- net Net-(J3-Pad3) renamed /U2+
- net Net-(J4-Pad2) renamed /U3-
- net Net-(J4-Pad3) renamed /U3+
Routing:
- net /D0+: track 69.1 -> 61.3 mm
- net /D0-: track 57.9 -> 51.0 mm
- net /U0+: track 11.9 -> 16.6 mm
- net /U0-: track 16.9 -> 19.8 mm
- net GND: track 133.1 -> 130.4 mm, vias 18 -> 27
- net VBUS: track 124.0 -> 121.3 mm
- net Net-(J1-Pad6): track 12.9 -> 15.2 mm
- net /U3-: track 26.8 -> 27.4 mm
- net /U3+: track 28.5 -> 29.2 mm
- net /U2-: track 30.8 -> 31.4 mm
- net /U2+: track 28.9 -> 29.6 mm
- net /U1-: track 26.0 -> 26.7 mm
- net /U1+: track 29.6 -> 30.2 mm
Other:
- board text added: "TUSB2036 USB Hub Evaluation Board v4 C. Keller 2021-04-14"
- board text removed: "TUSB2036 USB Hub Evaluation Board v3 C. Keller 2021-04-05"
